File: Roro1/eagle/HE6-RORO1.sch (EAGLE design)
At the start: 21 parts, among them U3 ESP32-WROOM-32(8MB)

Commit message: .
Parts:
- removed D1: WS2812B, SparkFun-LED:WS2812B
- removed IPEX: (no value), A-3-7-1-2-80:MICROBUILDER_ANTENNA_U.FL
- removed J2: (no value), SparkFun-Connectors:CONN_12NO_SILK
- removed S1, S2: MOMENTARY-SWITCH-SPST-SMD-6.0X3.5MM, SparkFun-Switches:MOMENTARY-SWITCH-SPST-SMD-6.0X3.5MM
- added ANT: (no value), A-3-7-1-2-80:MICROBUILDER_ANTENNA_U.FL
- added C1: 1nF, JLR:CAP0805
- added J3, J4: (no value), SparkFun-Connectors:CONN_14NO_SILK
- added NEO: WS2812B, SparkFun-LED:WS2812B
- added PGM, RST: MOMENTARY-SWITCH-SPST-SMD-6.0X3.5MM, SparkFun-Switches:MOMENTARY-SWITCH-SPST-SMD-6.0X3.5MM
- J1: device SparkFun-Connectors:CONN_12NO_SILK -> SparkFun-Connectors:CONN_01PTH_NO_SILK_YES_STOP
Connections:
- removed net BAT+: D2.A, J1.1, R4.1
- removed net IO16: J1.6, U3.IO16
- removed net IO17: J1.7, U3.IO17
- removed net IO2: J2.1, U3.IO2
- new net DIO1: J3.3, U1.DIO1
- new net DIO2: J3.2, U1.DIO2
- new net DIO3: J4.1, U1.DIO3
- new net DIO4: J3.4, U1.DIO4
- new net IO13: J4.2, U3.IO13
- new net NEOPIXEL: NEO.DI, U3.IO2
- new net RXD2: J3.7, U3.IO17
- new net TXD2: J3.6, U3.IO16
- new net VBAT: C1.2, D2.A, J3.1, NEO.VDD, R4.1
- net +3V3: now also J3.12, J4.12; no longer J1.12
- net GND: now also ANT.GND@0, ANT.GND@1, C1.1, J3.11, J4.10, NEO.VSS, PGM.2, RST.1; no longer IPEX.GND@0, IPEX.GND@1, J2.4
- net IO12: now also J4.3; no longer J2.5
- net IO14: now also J4.4; no longer J2.6
- net IO15: now also J3.5; no longer J2.3
- net IO26: now also J4.6; no longer J2.8
- net IO27: now also J4.5; no longer J2.7
- net IO33: now also J4.7; no longer J2.9
- net MISO: now also J3.9
- net MOSI: now also J3.10
- net N$1: now also ANT.SIGNAL, J1.1; no longer IPEX.SIGNAL
- net PGM: now also PGM.1
- net RST: now also J4.11, RST.2; no longer J2.12
- net RXD0: now also J4.13; no longer J1.9
- net SCK: now also J3.8
- net SCL: now also J3.13; no longer J1.11
- net SDA: now also J3.14; no longer J1.8
- net TXD0: now also J4.14; no longer J1.10
- net VN: now also J4.8; no longer J2.10
- net VP: now also J4.9; no longer J2.11
Other:
- note added: "STATUS INDICATION"
- moved on the sheet: C12, C2, D2, R1, R4, R5, R9

Commit message: .
Parts:
- PGM, RST: value MOMENTARY-SWITCH-SPST-SMD-6.0X3.5MM -> MOMENTARY-SWITCH-SPST-SMD-RIGHT-ANGLE; device SparkFun-Switches:MOMENTARY-SWITCH-SPST-SMD-6.0X3.5MM -> SparkFun-Switches:MOMENTARY-SWITCH-SPST-SMD-RIGHT-ANGLE
Connections:
- net RXD2: now also U3.IO16; no longer U3.IO17
- net TXD2: now also U3.IO17; no longer U3.IO16
Changed lines of the file:
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@@
 <part name="+3V1" library="supply1" deviceset="+3V3" device=""/>
 <part name="NEO" library="SparkFun-LED" library_urn="urn:adsk.eagle:library:529" deviceset="WS2812B" device="" package3d_urn="urn:adsk.eagle:package:39369/1" value="WS2812B"/>
-<part name="RST" library="SparkFun-Switches" library_urn="urn:adsk.eagle:library:535" deviceset="MOMENTARY-SWITCH-SPST" device="-SMD-6.0X3.5MM" package3d_urn="urn:adsk.eagle:package:40165/1" value="MOMENTARY-SWITCH-SPST-SMD-6.0X3.5MM"/>
-<part name="PGM" library="SparkFun-Switches" library_urn="urn:adsk.eagle:library:535" deviceset="MOMENTARY-SWITCH-SPST" device="-SMD-6.0X3.5MM" package3d_urn="urn:adsk.eagle:package:40165/1" value="MOMENTARY-SWITCH-SPST-SMD-6.0X3.5MM"/>
+<part name="RST" library="SparkFun-Switches" library_urn="urn:adsk.eagle:library:535" deviceset="MOMENTARY-SWITCH-SPST" device="-SMD-RIGHT-ANGLE" package3d_urn="urn:adsk.eagle:package:40169/1" value="MOMENTARY-SWITCH-SPST-SMD-RIGHT-ANGLE"/>
+<part name="PGM" library="SparkFun-Switches" library_urn="urn:adsk.eagle:library:535" deviceset="MOMENTARY-SWITCH-SPST" device="-SMD-RIGHT-ANGLE" package3d_urn="urn:adsk.eagle:package:40169/1" value="MOMENTARY-SWITCH-SPST-SMD-RIGHT-ANGLE"/>
 <part name="U$2" library="microbuilder" deviceset="VBAT" device=""/>
 <part name="GND2" library="supply1" deviceset="GND" device=""/>
@@
 <net name="TXD2" class="0">
 <segment>
+<pinref part="J3" gate="G$1" pin="6"/>
+<wire x1="99.06" y1="48.26" x2="101.6" y2="48.26" width="0.1524" layer="91"/>
+<label x="101.6" y="48.26" size="1.27" layer="95" xref="yes"/>
+</segment>
+<segment>
+<pinref part="U3" gate="G$1" pin="IO17"/>
+<wire x1="210.82" y1="119.38" x2="213.36" y2="119.38" width="0.1524" layer="91"/>
+<label x="213.36" y="119.38" size="1.27" layer="95" xref="yes"/>
+</segment>
+</net>
+<net name="RXD2" class="0">
+<segment>
+<pinref part="J3" gate="G$1" pin="7"/>
+<wire x1="99.06" y1="50.8" x2="101.6" y2="50.8" width="0.1524" layer="91"/>
+<label x="101.6" y="50.8" size="1.27" layer="95" xref="yes"/>
+</segment>
+<segment>
 <pinref part="U3" gate="G$1" pin="IO16"/>
 <wire x1="210.82" y1="121.92" x2="213.36" y2="121.92" width="0.1524" layer="91"/>
 <label x="213.36" y="121.92" size="1.27" layer="95" xref="yes"/>
 </segment>
-<segment>
-<pinref part="J3" gate="G$1" pin="6"/>
-<wire x1="99.06" y1="48.26" x2="101.6" y2="48.26" width="0.1524" layer="91"/>
-<label x="101.6" y="48.26" size="1.27" layer="95" xref="yes"/>
-</segment>
-</net>
-<net name="RXD2" class="0">
-<segment>
-<pinref part="U3" gate="G$1" pin="IO17"/>
-<wire x1="210.82" y1="119.38" x2="213.36" y2="119.38" width="0.1524" layer="91"/>
-<label x="213.36" y="119.38" size="1.27" layer="95" xref="yes"/>
-</segment>
-<segment>
-<pinref part="J3" gate="G$1" pin="7"/>
-<wire x1="99.06" y1="50.8" x2="101.6" y2="50.8" width="0.1524" layer="91"/>
-<label x="101.6" y="50.8" size="1.27" layer="95" xref="yes"/>
-</segment>
-</net>
+</net>
